File: USB to UART Converter.kicad_sch (KiCad schematic)
At the start: 0 parts

Commit message: Added all the Components to Schematic Editor
Parts:
- added C1, C2, C3, C4: C, symbol Device:C
- added D1, D2: LED, symbol Device:LED
- added D3, D4, D5: LESD5D5.0CT1G, LESD5D50CT1G, symbol LESD5D5_0CT1G:LESD5D5.0CT1G
- added J1: USB_C_Receptacle_USB2.0_16P, symbol Connector:USB_C_Receptacle_USB2.0_16P
- added J2: Conn_01x05_Pin, symbol Connector:Conn_01x05_Pin
- added R1, R2, R3, R4, R5, R6, R7: R, symbol Device:R
- added U1: CP2102N-Axx-xQFN28, Package_DFN_QFN:QFN-28-1EP_5x5mm_P0.5mm_EP3.35x3.35mm, symbol Interface_USB:CP2102N-Axx-xQFN28
Connections:
- new net: U1.29 (GND), U1.3 (GND)
- new net: J1.A1 (GND), J1.A12 (GND), J1.B1 (GND), J1.B12 (GND)
- new net: J1.A4 (VBUS), J1.A9 (VBUS), J1.B4 (VBUS), J1.B9 (VBUS)
Other:
- title: (none) -> USB to UART Converter Project
